File: pcb/ai_breakout_ft2323RL.brd (EAGLE design)
At the start: 25.4 x 16.3 mm, 12 parts

Commit message: Revision 1.1
Parts:
- removed R3: 125, Ai_Passives:0603-RES
- removed U$2: FT2332RL, Ai_IC:SSOP28-LD
- added IC1: FT2332RL, Ai_IC:SSOP28-LD
- added R2: 125, Ai_Passives:RES-0603
- added U$3: AI-LOGOL, Ai_Miscellany:AI-LOGO-L
- C1, C2: device Ai_Passives:0603-CAP -> Ai_Passives:CAP-0603
- C3: device Ai_Passives:EIA3216 -> Ai_Passives:CAP-POL-EIA3216
- JP1: value M06X1 -> 1X06LONG
- JP2: value M04X1 -> 1X04
- R1: value (none) -> 1K; device Ai_Passives:0603-RES -> Ai_Passives:RES-0603
- USB1: value USB-MICROB -> USBMICROB
- moved C2 0.18 mm to (17.2, 14.8)
- moved JP1 0.13 mm to (6.30, 8.12)
- moved C1 0.13 mm to (13.8, 14.8)
- moved C3 0.12 mm to (16.1, 10.4)
- moved USB1 0.06 mm to (22.6, 8.89)
- renumbered LED1 to TXLED, LED2 to RXLED, LED3 to ON, U$1 to JP2
Connections:
- removed net N$9: ON.A, R3.2
- new net N$5: ON.A, R2.2
- net 3V3: now also IC1.17; no longer U$2.17
- net 5V: now also IC1.20; no longer U$2.20
- net CTS: now also IC1.11; no longer U$2.11
- net DTR: now also IC1.2; no longer U$2.2
- net GND: now also IC1.18, IC1.21, IC1.25, IC1.26, IC1.7; no longer U$2.18, U$2.21, U$2.25, U$2.26, U$2.7
- net N$1: now also IC1.23; no longer U$2.23
- net N$2: now also IC1.22; no longer U$2.22
- net N$3: now also IC1.16; no longer U$2.16
- net N$4: now also IC1.15; no longer U$2.15
- net PWR: now also IC1.4, R2.1; no longer R3.1, U$2.4
- net RXI: now also IC1.5; no longer U$2.5
- net TXO: now also IC1.1; no longer U$2.1
Routing:
- net 5V: track 37.7 -> 46.8 mm, vias 2 -> 1
- net GND: track 18.5 -> 14.3 mm, vias 2 -> 4
- net DTR: track 14.9 -> 12.4 mm, vias 1 -> 0
- net RXI: track 14.1 -> 12.1 mm
- net N$5: track 0.00 -> 1.43 mm
- net N$9: track 1.31 -> 0.00 mm
- net N$1: track 9.13 -> 9.63 mm
Other:
- board text added: "JUMPER SETS PWR TO 3V3/5V"
- board text added: "VCC"
- board text added: "http://acrobotic.com"
- board text added: "v1.1"
- board text removed: "C3"
- board text removed: "ON"

Commit message: Finalized BOM
Parts:
- removed JP2: 1X04, Ai_Connectors:1X04
- added J1: 1X06LONG, Ai_Connectors:1X06-LONG
- JP1: value 1X06LONG -> 1X04-PJ; device Ai_Connectors:1X06-LONG -> Ai_Connectors:1X04
- R1: value 1K -> 300
- R2: value 125 -> 1K
- moved JP1 15.2 mm to (20.0, 1.45), turned to 0 degrees
Connections:
- net 3V3: now also JP1.4; no longer JP2.4
- net 5V: now also JP1.1; no longer JP2.1
- net CTS: now also J1.2; no longer JP1.2
- net DTR: now also J1.6; no longer JP1.6
- net GND: now also J1.1; no longer JP1.1
- net PWR: now also J1.3, JP1.2; no longer JP2.2, JP2.3
- net RXI: now also J1.5; no longer JP1.5
- net TXO: now also J1.4; no longer JP1.4
Changed lines of the file:
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@@
 </autorouter>
 <elements>
-<element name="JP1" library="Ai_Connectors" package="1X06-LONG" value="1X06LONG" x="6.3" y="8.123" smashed="yes" rot="R90"/>
-<element name="JP2" library="Ai_Connectors" package="1X04" value="1X04" x="20" y="1.45" smashed="yes"/>
+<element name="J1" library="Ai_Connectors" package="1X06-LONG" value="1X06LONG" x="6.3" y="8.123" smashed="yes" rot="R90"/>
+<element name="JP1" library="Ai_Connectors" package="1X04" value="1X04-PJ" x="20" y="1.45" smashed="yes"/>
 <element name="C1" library="Ai_Passives" package="CAP-0603" value="0.1uF" x="13.8" y="14.823" smashed="yes" rot="R180">
 <attribute name="NAME" x="12.065" y="13.335" size="0.762" layer="25" font="vector" ratio="15"/>
@@
 <attribute name="NAME" x="18.288" y="13.335" size="0.762" layer="25" font="vector" ratio="15"/>
 </element>
-<element name="R1" library="Ai_Passives" package="RES-0603" value="1K" x="22.55" y="5.5" smashed="yes" rot="R270">
+<element name="R1" library="Ai_Passives" package="RES-0603" value="300" x="22.55" y="5.5" smashed="yes" rot="R270">
 <attribute name="NAME" x="21.844" y="5.08" size="0.762" layer="25" font="vector" ratio="15" rot="R90"/>
 </element>
-<element name="R2" library="Ai_Passives" package="RES-0603" value="125" x="13.255" y="1.32" smashed="yes">
+<element name="R2" library="Ai_Passives" package="RES-0603" value="1K" x="13.255" y="1.32" smashed="yes">
 <attribute name="NAME" x="11.557" y="1.016" size="0.762" layer="25" font="vector" ratio="15" rot="R180"/>
 </element>
@@
 <via x="11.049" y="2.159" extent="1-16" drill="0.508"/>
 <via x="19.685" y="6.477" extent="1-16" drill="0.508"/>
-<contactref element="JP1" pad="1"/>
+<contactref element="J1" pad="1"/>
 <wire x1="6.3" y1="1.773" x2="10.663" y2="1.773" width="0.254" layer="16"/>
 <wire x1="10.663" y1="1.773" x2="11.049" y2="2.159" width="0.254" layer="16"/>
@@
 </signal>
 <signal name="5V">
-<contactref element="JP2" pad="1"/>
+<contactref element="JP1" pad="1"/>
 <contactref element="C1" pad="1"/>
 <contactref element="R1" pad="2"/>
@@
 </signal>
 <signal name="3V3">
-<contactref element="JP2" pad="4"/>
+<contactref element="JP1" pad="4"/>
 <contactref element="C2" pad="1"/>
 <wire x1="24.1532" y1="3.454" x2="24.1532" y2="14.5818" width="0.254" layer="16"/>
@@
 <signal name="TXO">
 <contactref element="IC1" pad="1"/>
-<contactref element="JP1" pad="4"/>
+<contactref element="J1" pad="4"/>
 <wire x1="6.3" y1="9.393" x2="7.371" y2="9.393" width="0.254" layer="1"/>
 <wire x1="7.371" y1="9.393" x2="10.922" y2="5.715" width="0.254" layer="1"/>
@@
 <signal name="CTS">
 <contactref element="IC1" pad="11"/>
-<contactref element="JP1" pad="2"/>
+<contactref element="J1" pad="2"/>
 <wire x1="6.3" y1="4.313" x2="7.371" y2="4.313" width="0.254" layer="16"/>
 <wire x1="7.371" y1="4.313" x2="8.509" y2="3.175" width="0.254" layer="16"/>
@@
 <signal name="RXI">
 <contactref element="IC1" pad="5"/>
-<contactref element="JP1" pad="5"/>
+<contactref element="J1" pad="5"/>
 <via x="13.97" y="6.35" extent="1-16" drill="0.508"/>
 <wire x1="9.017" y1="11.938" x2="6.305" y2="11.938" width="0.254" layer="16"/>
@@
 <signal name="DTR">
 <contactref element="IC1" pad="2"/>
-<contactref element="JP1" pad="6"/>
+<contactref element="J1" pad="6"/>
 <wire x1="6.3" y1="14.473" x2="7.244" y2="14.473" width="0.254" layer="1"/>
 <wire x1="7.244" y1="14.473" x2="9.5885" y2="12.2555" width="0.254" layer="1"/>
@@
 </signal>
 <signal name="PWR">
+<contactref element="J1" pad="3"/>
 <contactref element="JP1" pad="3"/>
-<contactref element="JP2" pad="3"/>
-<contactref element="JP2" pad="2"/>
+<contactref element="JP1" pad="2"/>
 <contactref element="R2" pad="1"/>
 <via x="17.2008" y="7.2524" extent="1-16" drill="0.508" diameter="0.254"/>
