File: pcb/ai_breakout_ft2323RL.sch (EAGLE design)
At the start: 12 parts

Commit message: Revision 1.1
Parts:
- removed LED1, LED2: YELLOW, Ai_LED:LED-0603
- removed LED3: BLUE, Ai_LED:LED-0603
- removed R3: 125, Ai_Passives:RES
- removed U$1: M04X1, Ai_Connectors:M04X1
- removed U$2: FT2332RL, Ai_IC:FT2332RL
- added IC1: FT2332RL, Ai_IC:FT2332RL
- added JP2: 1X04, Ai_Connectors:1X04
- added ON: BLUE, Ai_LED:LED0603
- added R2: 125, Ai_Passives:RES0603
- added RXLED, TXLED: YELLOW, Ai_LED:LED0603
- added U$3: AI-LOGOL, Ai_Miscellany:AI-LOGOL
- C1, C2: device Ai_Passives:CAP -> Ai_Passives:CAP0603
- C3: device Ai_Passives:CAP_POL -> Ai_Passives:CAP-POLEIA3216
- JP1: value M06X1 -> 1X06LONG; device Ai_Connectors:M06X1 -> Ai_Connectors:1X06LONG
- R1: value (none) -> 1K; device Ai_Passives:RES -> Ai_Passives:RES0603
- USB1: value USB-MICROB -> USBMICROB; device Ai_Connectors:USB-MICROB -> Ai_Connectors:USBMICROB
Connections:
- removed net N$9: LED3.A, R3.2
- new net N$5: ON.A, R2.2
- net 3V3: now also IC1.3V3OUT, JP2.4; no longer U$1.4, U$2.3V3OUT
- net 5V: now also C3.A, IC1.VCC, JP2.1; no longer C3.+, U$1.1, U$2.VCC
- net CTS: now also IC1.!CTS; no longer U$2.CTS
- net DTR: now also IC1.!DTR; no longer U$2.DTR
- net GND: now also C3.C, IC1.AGND, IC1.GND@1, IC1.GND@2, IC1.GND@3, IC1.TEST, ON.C; no longer C3.-, LED3.C, U$2.AGND, U$2.GND18, U$2.GND21, U$2.GND7, U$2.TEST
- net N$1: now also IC1.!TXLED, TXLED.C; no longer LED1.C, U$2.TXLED
- net N$2: now also IC1.!RXLED, RXLED.C; no longer LED2.C, U$2.RXLED
- net N$3: now also IC1.USBDM; no longer U$2.USBDM
- net N$4: now also IC1.USBDP; no longer U$2.USBDP
- net N$6: now also RXLED.A, TXLED.A; no longer LED1.A, LED2.A
- net PWR: now also IC1.VCCIO, JP2.2, JP2.3, R2.1; no longer R3.1, U$1.2, U$1.3, U$2.VCCIO
- net RXI: now also IC1.RXD; no longer U$2.RXD
- net TXO: now also IC1.TXD; no longer U$2.TXD
Other:
- moved on the sheet: C1, C2, R1

Commit message: Finalized BOM
Parts:
- removed JP2: 1X04, Ai_Connectors:1X04
- added J1: 1X06LONG, Ai_Connectors:1X06LONG
- JP1: value 1X06LONG -> 1X04-PJ; device Ai_Connectors:1X06LONG -> Ai_Connectors:1X04-PJ
- R1: value 1K -> 300
- R2: value 125 -> 1K
Connections:
- net 3V3: now also JP1.4; no longer JP2.4
- net 5V: now also JP1.1; no longer JP2.1
- net CTS: now also J1.2; no longer JP1.2
- net DTR: now also J1.6; no longer JP1.6
- net GND: now also J1.1; no longer JP1.1
- net PWR: now also J1.3, JP1.2; no longer JP2.2, JP2.3
- net RXI: now also J1.5; no longer JP1.5
- net TXO: now also J1.4; no longer JP1.4
Changed lines of the file:
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@@
 <attribute name="REV" value="1.1"/>
 </part>
-<part name="JP1" library="Ai_Connectors" deviceset="1X06" device="LONG"/>
-<part name="JP2" library="Ai_Connectors" deviceset="1X04" device=""/>
+<part name="J1" library="Ai_Connectors" deviceset="1X06" device="LONG"/>
+<part name="JP1" library="Ai_Connectors" deviceset="1X04-PJ" device=""/>
 <part name="C1" library="Ai_Passives" deviceset="CAP" device="0603" value="0.1uF"/>
 <part name="C2" library="Ai_Passives" deviceset="CAP" device="0603" value="0.1uF"/>
-<part name="R1" library="Ai_Passives" deviceset="RES" device="0603" value="1K"/>
-<part name="R2" library="Ai_Passives" deviceset="RES" device="0603" value="125"/>
+<part name="R1" library="Ai_Passives" deviceset="RES" device="0603" value="300"/>
+<part name="R2" library="Ai_Passives" deviceset="RES" device="0603" value="1K"/>
 <part name="GND1" library="Ai_Power" deviceset="GND" device=""/>
 <part name="GND2" library="Ai_Power" deviceset="GND" device=""/>
@@
 <attribute name="REV" x="238.76" y="10.16" size="2.54" layer="94"/>
 </instance>
-<instance part="JP1" gate="M06X1" x="105.41" y="69.85" rot="R180"/>
-<instance part="JP2" gate="G$1" x="165.1" y="73.66" rot="R180"/>
+<instance part="J1" gate="M06X1" x="105.41" y="69.85" rot="R180"/>
+<instance part="JP1" gate="G$1" x="162.56" y="73.66" rot="R270"/>
 <instance part="C1" gate="G$1" x="88.9" y="115.57"/>
 <instance part="C2" gate="G$1" x="109.22" y="115.57"/>
@@
 </segment>
 <segment>
-<pinref part="JP1" gate="M06X1" pin="1"/>
+<pinref part="J1" gate="M06X1" pin="1"/>
 <wire x1="100.33" y1="77.47" x2="95.25" y2="77.47" width="0.1524" layer="91"/>
 <label x="95.25" y="77.47" size="1.27" layer="95" ratio="15" rot="R180" xref="yes"/>
@@
 <net name="5V" class="0">
 <segment>
-<pinref part="JP2" gate="G$1" pin="1"/>
+<pinref part="JP1" gate="G$1" pin="1"/>
 <wire x1="160.02" y1="78.74" x2="157.48" y2="78.74" width="0.1524" layer="91"/>
 <pinref part="U$6" gate="G$1" pin="5V"/>
@@
 <segment>
 <wire x1="160.02" y1="71.12" x2="153.67" y2="71.12" width="0.1524" layer="91"/>
-<pinref part="JP2" gate="G$1" pin="4"/>
+<pinref part="JP1" gate="G$1" pin="4"/>
 <pinref part="U$5" gate="G$1" pin="3V3"/>
 <wire x1="153.67" y1="71.12" x2="153.67" y2="80.01" width="0.1524" layer="91"/>
@@
 </segment>
 <segment>
-<pinref part="JP1" gate="M06X1" pin="4"/>
+<pinref part="J1" gate="M06X1" pin="4"/>
 <wire x1="100.33" y1="69.85" x2="95.25" y2="69.85" width="0.1524" layer="91"/>
 <label x="95.25" y="69.85" size="1.27" layer="95" ratio="15" rot="R180" xref="yes"/>
@@
 </segment>
 <segment>
-<pinref part="JP1" gate="M06X1" pin="2"/>
+<pinref part="J1" gate="M06X1" pin="2"/>
 <wire x1="100.33" y1="74.93" x2="95.25" y2="74.93" width="0.1524" layer="91"/>
 <label x="95.25" y="74.93" size="1.27" layer="95" ratio="15" rot="R180" xref="yes"/>
@@
 </segment>
 <segment>
-<pinref part="JP1" gate="M06X1" pin="5"/>
+<pinref part="J1" gate="M06X1" pin="5"/>
 <wire x1="100.33" y1="67.31" x2="95.25" y2="67.31" width="0.1524" layer="91"/>
 <label x="95.25" y="67.31" size="1.27" layer="95" ratio="15" rot="R180" xref="yes"/>
@@
 </segment>
 <segment>
-<pinref part="JP1" gate="M06X1" pin="6"/>
+<pinref part="J1" gate="M06X1" pin="6"/>
 <wire x1="100.33" y1="64.77" x2="95.25" y2="64.77" width="0.1524" layer="91"/>
 <label x="95.25" y="64.77" size="1.27" layer="95" ratio="15" rot="R180" xref="yes"/>
@@
 <net name="PWR" class="0">
 <segment>
-<pinref part="JP1" gate="M06X1" pin="3"/>
+<pinref part="J1" gate="M06X1" pin="3"/>
 <wire x1="100.33" y1="72.39" x2="97.79" y2="72.39" width="0.1524" layer="91"/>
 <wire x1="97.79" y1="72.39" x2="97.79" y2="80.01" width="0.1524" layer="91"/>
@@
 </segment>
 <segment>
-<pinref part="JP2" gate="G$1" pin="3"/>
+<pinref part="JP1" gate="G$1" pin="3"/>
 <wire x1="148.59" y1="73.66" x2="160.02" y2="73.66" width="0.1524" layer="91"/>
-<pinref part="JP2" gate="G$1" pin="2"/>
+<pinref part="JP1" gate="G$1" pin="2"/>
 <wire x1="148.59" y1="76.2" x2="160.02" y2="76.2" width="0.1524" layer="91"/>
 <wire x1="148.59" y1="73.66" x2="148.59" y2="74.93" width="0.1524" layer="91"/>
