File: pcb/ai_breakout_ft232RL.brd (EAGLE design)
At the start: 16.3 x 25.5 mm, 14 parts, among them IC1 FT2332RL, J1 1X06LONG

Commit message: updating libraries
Parts:
- JP1: value 1X04-PJ -> 1X04NOSILK; device Ai_Connectors:1X04 -> Ai_Connectors:1X04-NOSILK
Changed lines of the file:
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@@
 <?xml version="1.0" encoding="utf-8"?>
 <!DOCTYPE eagle SYSTEM "eagle.dtd">
-<eagle version="6.5.0">
+<eagle version="7.1.0">
 <drawing>
 <settings>
@@
 <setting verticaltext="up"/>
 </settings>
-<grid distance="5" unitdist="mil" unit="mil" style="lines" multiple="1" display="yes" altdistance="0.025" altunitdist="inch" altunit="inch"/>
+<grid distance="1" unitdist="mil" unit="mil" style="lines" multiple="1" display="yes" altdistance="0.025" altunitdist="inch" altunit="inch"/>
 <layers>
 <layer number="1" name="Top" color="4" fill="1" visible="yes" active="yes"/>
@@
 <layer number="97" name="Info" color="7" fill="1" visible="no" active="no"/>
 <layer number="98" name="Guide" color="6" fill="1" visible="no" active="no"/>
+<layer number="99" name="SpiceOrder" color="7" fill="1" visible="no" active="no"/>
 <layer number="100" name="Muster" color="7" fill="1" visible="no" active="no"/>
 <layer number="101" name="Patch_Top" color="12" fill="4" visible="no" active="yes"/>
@@
 <pass name="Default">
 <param name="RoutingGrid" value="10mil"/>
+<param name="AutoGrid" value="1"/>
+<param name="Efforts" value="0"/>
+<param name="TopRouterVariant" value="1"/>
 <param name="tpViaShape" value="round"/>
 <param name="PrefDir.1" value="*"/>
@@
 <elements>
 <element name="J1" library="Ai_Connectors" package="1X06-LONG" value="1X06LONG" x="8.133" y="21.032" smashed="yes" rot="R180"/>
-<element name="JP1" library="Ai_Connectors" package="1X04" value="1X04-PJ" x="1.45" y="5.146" smashed="yes" rot="R270"/>
+<element name="JP1" library="Ai_Connectors" package="1X04-NOSILK" value="1X04NOSILK" x="1.45" y="5.146" smashed="yes" rot="R270"/>
 <element name="C1" library="Ai_Passives" package="CAP-0603" value="0.1uF" x="2.032" y="11.684" smashed="yes">
 <attribute name="NAME" x="3.81" y="11.049" size="0.762" layer="25" font="vector" ratio="15" rot="R180"/>
@@
 <contactref element="C3" pad="2"/>
 <contactref element="J1" pad="1"/>
-<wire x1="3.7" y1="10.866" x2="2.882" y2="11.684" width="0.4064" layer="1"/>
+<wire x1="3.7" y1="10.866" x2="2.932" y2="11.684" width="0.4064" layer="1"/>
 <via x="3.429" y="9.906" extent="1-16" drill="0.508"/>
 <via x="12.192" y="4.3434" extent="1-16" drill="0.508"/>
@@
 <wire x1="3.683" y1="5.588" x2="6.574" y2="5.588" width="0.4064" layer="1"/>
 <wire x1="6.574" y1="5.588" x2="6.828" y2="5.334" width="0.4064" layer="1"/>
-<wire x1="13.337" y1="9.566" x2="13.97" y2="10.199" width="0.4064" layer="1"/>
-<wire x1="12.358" y1="17.018" x2="9.232" y2="13.931" width="0.4064" layer="1"/>
+<wire x1="13.337" y1="9.566" x2="13.97" y2="10.149" width="0.4064" layer="1"/>
+<wire x1="12.308" y1="17.018" x2="9.232" y2="13.931" width="0.4064" layer="1"/>
 <wire x1="9.232" y1="13.931" x2="8.509" y2="13.208" width="0.4064" layer="1"/>
 <wire x1="8.509" y1="13.208" x2="8.509" y2="10.541" width="0.4064" layer="1"/>
 <wire x1="8.509" y1="10.541" x2="6.828" y2="8.86" width="0.4064" layer="1"/>
-<wire x1="1.182" y1="11.684" x2="1.182" y2="9.224" width="0.4064" layer="1"/>
-<wire x1="1.182" y1="9.224" x2="1.45" y2="8.956" width="0.4064" layer="1"/>
+<wire x1="1.132" y1="11.684" x2="1.1312" y2="9.2494" width="0.4064" layer="1"/>
+<wire x1="1.1312" y1="9.2494" x2="1.45" y2="8.956" width="0.4064" layer="1"/>
 <contactref element="IC1" pad="20"/>
 <wire x1="13.337" y1="9.566" x2="12.165" y2="9.566" width="0.4064" layer="1"/>
@@
 <contactref element="C2" pad="1"/>
 <wire x1="13.72" y1="7.616" x2="13.97" y2="7.366" width="0.4064" layer="1"/>
-<wire x1="13.97" y1="7.366" x2="13.97" y2="6.184" width="0.4064" layer="1"/>
+<wire x1="13.97" y1="7.366" x2="13.97" y2="6.234" width="0.4064" layer="1"/>
 <via x="15.367" y="1.778" extent="1-16" drill="0.508"/>
 <wire x1="15.367" y1="1.778" x2="15.367" y2="5.842" width="0.4064" layer="1"/>
 <wire x1="15.367" y1="5.842" x2="15.113" y2="6.096" width="0.4064" layer="1"/>
 <wire x1="15.113" y1="6.096" x2="14.058" y2="6.096" width="0.4064" layer="1"/>
-<wire x1="14.058" y1="6.096" x2="13.97" y2="6.184" width="0.4064" layer="1"/>
+<wire x1="14.058" y1="6.096" x2="13.97" y2="6.234" width="0.4064" layer="1"/>
 <contactref element="IC1" pad="17"/>
 <wire x1="13.72" y1="7.616" x2="12.165" y2="7.616" width="0.4064" layer="1"/>
@@
 <contactref element="R1" pad="1"/>
 <wire x1="15.494" y1="10.148" x2="15.494" y2="11.95" width="0.4064" layer="1"/>
-<wire x1="13.97" y1="11.899" x2="15.443" y2="11.899" width="0.4064" layer="1"/>
+<wire x1="13.97" y1="11.949" x2="15.443" y2="11.899" width="0.4064" layer="1"/>
 <wire x1="15.443" y1="11.899" x2="15.494" y2="11.95" width="0.4064" layer="1"/>
 </signal>
@@
 <contactref element="ON" pad="A"/>
 <wire x1="1.143" y1="14.974" x2="1.932" y2="14.974" width="0.4064" layer="1"/>
-<wire x1="1.932" y1="14.974" x2="2.667" y2="15.709" width="0.4064" layer="1"/>
+<wire x1="1.932" y1="14.974" x2="2.667" y2="15.759" width="0.4064" layer="1"/>
 </signal>
 <signal name="TXO">
@@
 <wire x1="3.683" y1="14.351" x2="3.683" y2="16.891" width="0.3048" layer="1"/>
 <wire x1="3.683" y1="16.891" x2="3.556" y2="17.018" width="0.3048" layer="1"/>
-<wire x1="3.556" y1="17.018" x2="2.882" y2="17.272" width="0.3048" layer="1"/>
+<wire x1="3.556" y1="17.018" x2="2.932" y2="17.272" width="0.3048" layer="1"/>
 <contactref element="IC1" pad="2"/>
 <wire x1="3.918" y1="14.116" x2="4.853" y2="14.116" width="0.3048" layer="1"/>
@@
 <wire x1="6.35" y1="6.858" x2="6.35" y2="13.335" width="0.4064" layer="16"/>
 <via x="6.35" y="13.335" extent="1-16" drill="0.508"/>
-<wire x1="2.667" y1="14.009" x2="2.755" y2="14.009" width="0.4064" layer="1"/>
+<wire x1="2.667" y1="13.959" x2="2.755" y2="14.009" width="0.4064" layer="1"/>
 <wire x1="2.755" y1="14.009" x2="3.948" y2="12.816" width="0.4064" layer="1"/>
 <wire x1="9.403" y1="21.032" x2="9.403" y2="20.198" width="0.4064" layer="1"/>
@@
 <contactref element="C4" pad="2"/>
 <contactref element="J1" pad="6"/>
-<wire x1="1.182" y1="17.272" x2="1.182" y2="20.431" width="0.3048" layer="1"/>
+<wire x1="1.132" y1="17.272" x2="1.182" y2="20.431" width="0.3048" layer="1"/>
 <wire x1="1.182" y1="20.431" x2="1.783" y2="21.032" width="0.3048" layer="1"/>
 </signal>
