File: pcb/ai_breakout_ft232RL.sch (EAGLE design)
At the start: 14 parts, among them IC1 FT2332RL, J1 1X06LONG

Commit message: updating libraries
Parts:
- JP1: value 1X04-PJ -> 1X04NOSILK; device Ai_Connectors:1X04-PJ -> Ai_Connectors:1X04NOSILK
Changed lines of the file:
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@@
 <?xml version="1.0" encoding="utf-8"?>
 <!DOCTYPE eagle SYSTEM "eagle.dtd">
-<eagle version="6.5.0">
+<eagle version="7.1.0">
 <drawing>
 <settings>
@@
 <setting verticaltext="up"/>
 </settings>
-<grid distance="0.1" unitdist="inch" unit="inch" style="lines" multiple="1" display="no" altdistance="0.01" altunitdist="inch" altunit="inch"/>
+<grid distance="50" unitdist="mil" unit="mil" style="lines" multiple="1" display="yes" altdistance="0.01" altunitdist="inch" altunit="inch"/>
 <layers>
 <layer number="1" name="Top" color="4" fill="1" visible="no" active="no"/>
@@
 <layer number="97" name="Info" color="7" fill="1" visible="yes" active="yes"/>
 <layer number="98" name="Guide" color="6" fill="1" visible="yes" active="yes"/>
+<layer number="99" name="SpiceOrder" color="7" fill="1" visible="yes" active="yes"/>
 <layer number="100" name="Muster" color="7" fill="1" visible="no" active="no"/>
 <layer number="101" name="Patch_Top" color="12" fill="4" visible="no" active="yes"/>
@@
 </part>
 <part name="J1" library="Ai_Connectors" deviceset="1X06" device="LONG"/>
-<part name="JP1" library="Ai_Connectors" deviceset="1X04-PJ" device=""/>
+<part name="JP1" library="Ai_Connectors" deviceset="1X04" device="NOSILK"/>
 <part name="C1" library="Ai_Passives" deviceset="CAP" device="0603" value="0.1uF"/>
 <part name="C2" library="Ai_Passives" deviceset="CAP" device="0603" value="0.1uF"/>
@@
 <instance part="FRAME1" gate="G$2" x="147.32" y="0"/>
 <instance part="J1" gate="M06X1" x="105.41" y="69.85" rot="R180"/>
-<instance part="JP1" gate="G$1" x="160.02" y="73.66" rot="R270"/>
+<instance part="JP1" gate="G$1" x="162.56" y="73.66" rot="R180"/>
 <instance part="C1" gate="G$1" x="88.9" y="115.57"/>
 <instance part="C2" gate="G$1" x="109.22" y="115.57"/>
